File: Hardware/PIC12_UNIVERSAL_Devboard_v1_THT/PIC12_UNIVERSAL_Devboard_v1_THT.kicad_sch (KiCad schematic)
At the start: 33 parts, among them J2 Conn_PIC_ICSP_ICD, J3 Screw_Terminal_01x02, J4 Conn_01x07_Pin, SW1 SW_RESET, U1 PIC12F617-xP, U2 78L05G-AB3-R, U3 XC6206-3.3V_C3015484

Commit message: PIC12 Universal Dev Board - Schematics - Added Reverse Current Protection PMOS for XC6240 Regulator
Signed-off-by: alexanderjg85 <alexanderjg85@gmail.com>
Parts:
- added R4: 10k, Resistor_SMD:R_1206_3216Metric_Pad1.30x1.75mm_HandSolder, symbol Device:R_Small
- added U4: SI2301-A1SHB, AJ_Transistors:C28642376_SOT-23-3_L2_9-W1_3-P1_90-LS2_4-BR, symbol AJ_Transistors:SI2301-A1SHB
Connections:
- net GND: now also R4.2
- net VCC_5: now also R4.1, U4.1 (G)
- net VDD: now also U4.2 (S); no longer C3.1, U3.2 (VOUT)
- new net: C3.1, U3.2 (VOUT), U4.3 (D)
Other:
- moved on the sheet: C3, C4, TP4, U3

Commit message: PIC12 Universal Dev Board - Schematics - Added Part Properties
Signed-off-by: alexanderjg85 <alexanderjg85@gmail.com>
Parts:
- C1, C2, C3, C4: Package (none) -> 0805; Spec (none) -> ±10% 50V
- C5: Package (none) -> 0805
- D1, D4: LCSC (none) -> C2480; Package (none) -> SMA; Spec (none) -> 30V 0.5A Schottky Diode
- D2: Package (none) -> 3 mm; Spec (none) -> LED GREEN
- D3: Package (none) -> 3 mm; Spec (none) -> LED YELLOW
- J2: Package (none) -> 2.54 mm 1x6; Spec (none) -> Male / THT/ Vertical
- J3: Package (none) -> 5.08mm 1x2; Spec (none) -> Horizontal
- J4: Package (none) -> 2.54 mm 1x7; Spec (none) -> Male / THT/ Vertical
- JP1, JP3: Package (none) -> 2.54 mm 1x2; Spec (none) -> Male / THT/ Vertical
- JP2: Package (none) -> 2.54 mm 1x3; Spec (none) -> Male / THT/ Vertical; now in the parts list
- R1, R2, R3, R4: Package (none) -> 1206; Spec (none) -> 1% 125 mW
- SW1: Package (none) -> 4.5 x 4.5 SMD; Spec (none) -> H=5.0mm Tactile
- TP2: now left out of the parts list
- U1: MFR PN (none) -> PIC12F17I/P; Package (none) -> PDIP-8; Spec (none) -> 8-Bit PIC 20 Mhz
- U2: Package (none) -> SOT-89-3; Spec (none) -> 5V 0.1 A
- U3: Package (none) -> SOT23; Spec (none) -> 3.3V 0.25A
- U4: MFR PN (none) -> SI2301-A1SHB; Package (none) -> SOT23; Spec (none) -> P-Mos 20V 2.3A

Commit message: PIC12 Universal Dev Board - Updated Reset Switch Footprint for better Handsoldering
Signed-off-by: alexanderjg85 <alexanderjg85@gmail.com>
Parts:
- SW1: footprint Button_Switch_SMD:SW_SPST_PTS647_Sx38 -> AJ_Electromechanical:SW_SPST_PTS647_Sx38_Handsolder; MFR PN (none) -> SWT0210-045026GSA; Spec H=5.0mm Tactile -> H=4.5mm Tactile
Changed lines of the file:
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@@
 			)
 		)
-		(property "Footprint" "Button_Switch_SMD:SW_SPST_PTS647_Sx38"
+		(property "Footprint" "AJ_Electromechanical:SW_SPST_PTS647_Sx38_Handsolder"
 			(at 252.73 123.19 0)
 			(hide yes)
@@
 			)
 		)
-		(property "Spec" "H=5.0mm Tactile"
+		(property "Spec" "H=4.5mm Tactile"
 			(at 252.73 128.27 0)
 			(hide yes)
@@
 			)
 		)
-		(property "MFR PN" ""
+		(property "MFR PN" "SWT0210-045026GSA"
 			(at 252.73 128.27 0)
 			(hide yes)
